Commit message: sync https://www.lejuhub.com/highlydynamic/kuavo-ros-control/commit/c5f376581c0e6365722431704dfa744ba10364ed

File: src/kuavo_assets/models/biped_s45/urdf/drake/biped_v3_arm.urdf (robot description, URDF)
Before this commit: robot biped_s45, 17 links, 16 joints
Joints:
- joint zarm_l1_joint: limit lower=-3.14159265358979 upper=1.5707963267949 effort=100.0 velocity=41.3433333333333 -> lower=-3.14159265358979 upper=0.01 effort=100.0 velocity=41.3433333333333
- joint zarm_r1_joint: limit lower=-3.14159265358979 upper=1.5707963267949 effort=100.0 velocity=41.3433333333333 -> lower=-3.14159265358979 upper=0.01 effort=100.0 velocity=41.3433333333333
